File: CrawlerProc_ver_02.sch (EAGLE design)
At the start: 57 parts, among them U1 MIC5335-SPYMT, U10 ECS-160-8, U11 ANTENNA, U12 ANTENNA-CHIP, U2 MIC5320-JGYML, U3 ITG-3200, U4 AT86RF231-ZU, U5 AT45DB321D, U6 ECS-2033, U8 ADXL345-LGA12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

Commit message: Updated with routing for SPI breakout
Connections:
- removed net N$2: PROC.SDO2/CN10/RG8, U5.SI
- removed net N$42: PROC.SCK2/CN8/RG6, U5.SCK
- removed net N$45: PROC.SDI2/CN9/RG7, U5.SO
- removed net PWM2L: PROC.PWM2L/RE2, U$1.1
- new net SCK2: PROC.PWM2L/RE2, PROC.SCK2/CN8/RG6, U$1.1, U5.SCK
- new net SDI2: PROC.SDI2/CN9/RG7, U$1.9, U5.SO
- new net SDO2: PROC.SDO2/CN10/RG8, U$1.11, U5.SI
Changed lines of the file:
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@@
-</segment>
-</net>
-<net name="N$45" class="0">
-<segment>
-<wire x1="68.58" y1="93.98" x2="40.64" y2="93.98" width="0.1524" layer="91"/>
-<pinref part="U5" gate="G$1" pin="SO"/>
-<pinref part="PROC" gate="G$1" pin="SDI2/CN9/RG7"/>
 </segment>
 </net>
@@
 <label x="246.38" y="76.2" size="1.778" layer="95"/>
 <pinref part="JP2" gate="G$1" pin="HREF"/>
-</segment>
-</net>
-<net name="N$42" class="0">
-<segment>
-<wire x1="12.7" y1="91.44" x2="15.24" y2="91.44" width="0.1524" layer="91"/>
-<wire x1="12.7" y1="91.44" x2="12.7" y2="101.6" width="0.1524" layer="91"/>
-<wire x1="12.7" y1="101.6" x2="48.26" y2="101.6" width="0.1524" layer="91"/>
-<wire x1="48.26" y1="101.6" x2="48.26" y2="96.52" width="0.1524" layer="91"/>
-<wire x1="48.26" y1="96.52" x2="68.58" y2="96.52" width="0.1524" layer="91"/>
-<pinref part="U5" gate="G$1" pin="SCK"/>
-<pinref part="PROC" gate="G$1" pin="SCK2/CN8/RG6"/>
 </segment>
 </net>
@@
 <pinref part="R9" gate="G$1" pin="1"/>
 <pinref part="JP3" gate="G$1" pin="5"/>
-</segment>
-</net>
-<net name="N$2" class="0">
-<segment>
-<wire x1="45.72" y1="99.06" x2="15.24" y2="99.06" width="0.1524" layer="91"/>
-<wire x1="15.24" y1="99.06" x2="15.24" y2="93.98" width="0.1524" layer="91"/>
-<wire x1="45.72" y1="99.06" x2="45.72" y2="91.44" width="0.1524" layer="91"/>
-<wire x1="45.72" y1="91.44" x2="68.58" y2="91.44" width="0.1524" layer="91"/>
-<pinref part="U5" gate="G$1" pin="SI"/>
-<pinref part="PROC" gate="G$1" pin="SDO2/CN10/RG8"/>
 </segment>
 </net>
@@
 </segment>
 </net>
-<net name="PWM2L" class="0">
+<net name="SCK2" class="0">
 <segment>
 <wire x1="99.06" y1="124.46" x2="99.06" y2="127" width="0.1524" layer="91"/>
@@
 </segment>
 <segment>
-<wire x1="127" y1="187.96" x2="121.92" y2="187.96" width="0.2032" layer="91"/>
+<wire x1="127" y1="187.96" x2="124.46" y2="187.96" width="0.2032" layer="91"/>
 <label x="116.84" y="187.96" size="1.778" layer="95"/>
 <pinref part="U$1" gate="G$1" pin="1"/>
+<wire x1="124.46" y1="187.96" x2="121.92" y2="187.96" width="0.2032" layer="91"/>
+</segment>
+<segment>
+<wire x1="12.7" y1="91.44" x2="15.24" y2="91.44" width="0.1524" layer="91"/>
+<wire x1="12.7" y1="91.44" x2="12.7" y2="101.6" width="0.1524" layer="91"/>
+<wire x1="12.7" y1="101.6" x2="48.26" y2="101.6" width="0.1524" layer="91"/>
+<wire x1="48.26" y1="101.6" x2="48.26" y2="96.52" width="0.1524" layer="91"/>
+<wire x1="48.26" y1="96.52" x2="68.58" y2="96.52" width="0.1524" layer="91"/>
+<pinref part="U5" gate="G$1" pin="SCK"/>
+<pinref part="PROC" gate="G$1" pin="SCK2/CN8/RG6"/>
 </segment>
 </net>
@@
 </segment>
 </net>
+<net name="SDI2" class="0">
+<segment>
+<pinref part="U$1" gate="G$1" pin="9"/>
+<wire x1="127" y1="177.8" x2="121.92" y2="177.8" width="0.1524" layer="91"/>
+<label x="116.84" y="177.8" size="1.778" layer="95"/>
+</segment>
+<segment>
+<wire x1="68.58" y1="93.98" x2="40.64" y2="93.98" width="0.1524" layer="91"/>
+<pinref part="U5" gate="G$1" pin="SO"/>
+<pinref part="PROC" gate="G$1" pin="SDI2/CN9/RG7"/>
+</segment>
+</net>
+<net name="SDO2" class="0">
+<segment>
+<pinref part="U$1" gate="G$1" pin="11"/>
+<wire x1="127" y1="175.26" x2="121.92" y2="175.26" width="0.1524" layer="91"/>
+<label x="116.84" y="175.26" size="1.778" layer="95"/>
+<label x="116.84" y="175.26" size="1.778" layer="95"/>
+</segment>
+<segment>
+<wire x1="45.72" y1="99.06" x2="15.24" y2="99.06" width="0.1524" layer="91"/>
+<wire x1="15.24" y1="99.06" x2="15.24" y2="93.98" width="0.1524" layer="91"/>
+<wire x1="45.72" y1="99.06" x2="45.72" y2="91.44" width="0.1524" layer="91"/>
+<wire x1="45.72" y1="91.44" x2="68.58" y2="91.44" width="0.1524" layer="91"/>
+<pinref part="U5" gate="G$1" pin="SI"/>
+<pinref part="PROC" gate="G$1" pin="SDO2/CN10/RG8"/>
+</segment>
+</net>

Commit message: SPI breakout routing changes and Freerouter script
Changed lines of the file:
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@@
 <pinref part="U5" gate="G$1" pin="SCK"/>
 <pinref part="PROC" gate="G$1" pin="SCK2/CN8/RG6"/>
+<label x="60.96" y="96.52" size="1.778" layer="95"/>
 </segment>
 </net>
@@
 <segment>
 <pinref part="U$1" gate="G$1" pin="9"/>
-<wire x1="127" y1="177.8" x2="121.92" y2="177.8" width="0.1524" layer="91"/>
+<wire x1="127" y1="177.8" x2="121.92" y2="177.8" width="0.2032" layer="91"/>
 <label x="116.84" y="177.8" size="1.778" layer="95"/>
 </segment>
@@
 <pinref part="U5" gate="G$1" pin="SO"/>
 <pinref part="PROC" gate="G$1" pin="SDI2/CN9/RG7"/>
+<label x="60.96" y="93.98" size="1.778" layer="95"/>
 </segment>
 </net>
@@
 <segment>
 <pinref part="U$1" gate="G$1" pin="11"/>
-<wire x1="127" y1="175.26" x2="121.92" y2="175.26" width="0.1524" layer="91"/>
+<wire x1="127" y1="175.26" x2="121.92" y2="175.26" width="0.2032" layer="91"/>
 <label x="116.84" y="175.26" size="1.778" layer="95"/>
 <label x="116.84" y="175.26" size="1.778" layer="95"/>
